Commit message: Fixed Examples

File: assets/examples/complex-hexapod/complex-hexapod.urdf (robot description, URDF)
Before this commit: robot atlas_hexapod, 27 links, 26 joints
Links:
- removed link sensor_tower
- removed link stereo_camera
- added link lidar_link, mass 0.28; collision cylinder length=0.084 radius=0.07; visual cylinder length=0.038 radius=0.058
- added link sensor_pan_link, mass 0.65; collision cylinder length=0.16 radius=0.08; visual box size=0.11 0.25 0.07
- added link stereo_camera_link, mass 0.32; collision box size=0.12 0.28 0.10; visual box size=0.12 0.28 0.10
- link body_link: mass 14.5 -> 12.5; geometry collision box size=1.0 0.52 0.28; visual box size=0.08 0.42 0.18
- link front_left_coxa: mass 0.38 -> 0.45; geometry collision box size=0.22 0.10 0.09; visual box size=0.22 0.10 0.09
- link front_left_femur: mass 0.72 -> 0.75; geometry collision box size=0.40 0.12 0.11; visual box size=0.28 0.128 0.025
- link front_left_foot: mass 0.11 -> 0.12; geometry collision sphere radius=0.055; visual sphere radius=0.055
- link front_left_tibia: mass 0.58 -> 0.55; geometry collision box size=0.42 0.085 0.085; visual box size=0.22 0.092 0.018
- link front_right_coxa: mass 0.38 -> 0.45; geometry collision box size=0.22 0.10 0.09; visual box size=0.22 0.10 0.09
- link front_right_femur: mass 0.72 -> 0.75; geometry collision box size=0.40 0.12 0.11; visual box size=0.28 0.128 0.025
- link front_right_foot: mass 0.11 -> 0.12; geometry collision sphere radius=0.055; visual sphere radius=0.055
- link front_right_tibia: mass 0.58 -> 0.55; geometry collision box size=0.42 0.085 0.085; visual box size=0.22 0.092 0.018
- link middle_left_coxa: mass 0.38 -> 0.45; geometry collision box size=0.22 0.10 0.09; visual box size=0.22 0.10 0.09
- link middle_left_femur: mass 0.72 -> 0.75; geometry collision box size=0.40 0.12 0.11; visual box size=0.28 0.128 0.025
- link middle_left_foot: mass 0.11 -> 0.12; geometry collision sphere radius=0.055; visual sphere radius=0.055
- link middle_left_tibia: mass 0.58 -> 0.55; geometry collision box size=0.42 0.085 0.085; visual box size=0.22 0.092 0.018
- link middle_right_coxa: mass 0.38 -> 0.45; geometry collision box size=0.22 0.10 0.09; visual box size=0.22 0.10 0.09
- link middle_right_femur: mass 0.72 -> 0.75; geometry collision box size=0.40 0.12 0.11; visual box size=0.28 0.128 0.025
- link middle_right_foot: mass 0.11 -> 0.12; geometry collision sphere radius=0.055; visual sphere radius=0.055
- link middle_right_tibia: mass 0.58 -> 0.55; geometry collision box size=0.42 0.085 0.085; visual box size=0.22 0.092 0.018
- link rear_left_coxa: mass 0.38 -> 0.45; geometry collision box size=0.22 0.10 0.09; visual box size=0.22 0.10 0.09
- link rear_left_femur: mass 0.72 -> 0.75; geometry collision box size=0.40 0.12 0.11; visual box size=0.28 0.128 0.025
- link rear_left_foot: mass 0.11 -> 0.12; geometry collision sphere radius=0.055; visual sphere radius=0.055
- link rear_left_tibia: mass 0.58 -> 0.55; geometry collision box size=0.42 0.085 0.085; visual box size=0.22 0.092 0.018
- link rear_right_coxa: mass 0.38 -> 0.45; geometry collision box size=0.22 0.10 0.09; visual box size=0.22 0.10 0.09
- link rear_right_femur: mass 0.72 -> 0.75; geometry collision box size=0.40 0.12 0.11; visual box size=0.28 0.128 0.025
- link rear_right_foot: mass 0.11 -> 0.12; geometry collision sphere radius=0.055; visual sphere radius=0.055
- link rear_right_tibia: mass 0.58 -> 0.55; geometry collision box size=0.42 0.085 0.085; visual box size=0.22 0.092 0.018
Joints:
- removed joint front_left_ankle
- removed joint front_right_ankle
- removed joint middle_left_ankle
- removed joint middle_right_ankle
- removed joint rear_left_ankle
- removed joint rear_right_ankle
- removed joint sensor_tower_joint
- added joint front_left_foot_joint: type fixed, parent front_left_tibia, child front_left_foot, origin xyz=0.42 0 0 rpy=0 0 0
- added joint front_right_foot_joint: type fixed, parent front_right_tibia, child front_right_foot, origin xyz=0.42 0 0
- added joint lidar_joint: type continuous, parent body_link, child lidar_link, origin xyz=-0.27 0 0.93 rpy=0 0 0, axis 0 0 1, limit effort=2 velocity=8
- added joint middle_left_foot_joint: type fixed, parent middle_left_tibia, child middle_left_foot, origin xyz=0.42 0 0 rpy=0 0 0
- added joint middle_right_foot_joint: type fixed, parent middle_right_tibia, child middle_right_foot, origin xyz=0.42 0 0
- added joint rear_left_foot_joint: type fixed, parent rear_left_tibia, child rear_left_foot, origin xyz=0.42 0 0
- added joint rear_right_foot_joint: type fixed, parent rear_right_tibia, child rear_right_foot, origin xyz=0.42 0 0
- added joint sensor_pan_joint: type continuous, parent body_link, child sensor_pan_link, origin xyz=0.19 0 0.93 rpy=0 0 0, axis 0 0 1, limit effort=6 velocity=2.5
- joint camera_tilt_joint: child stereo_camera -> stereo_camera_link; limit lower=-0.9 upper=0.55 effort=5 velocity=2 -> lower=-0.95 upper=0.55 effort=5 velocity=2; origin xyz=0.1 0 0.25 rpy=0 0 0 -> xyz=0.07 0 0.16 rpy=0 0 0; parent sensor_tower -> sensor_pan_link
- joint front_left_hip_pitch: axis 1 0 0 -> 0 1 0; limit lower=-1.15 upper=1.15 effort=34 velocity=3 -> lower=-0.85 upper=1.05 effort=38 velocity=3; origin xyz=0 0.2 0 rpy=0 0 0 -> xyz=0.22 0 0 rpy=0 0.52 0
- joint front_left_hip_yaw: limit lower=-0.8 upper=0.8 effort=28 velocity=3 -> lower=-0.75 upper=0.75 effort=30 velocity=3; origin xyz=0.46 0.3 0 rpy=0 0 0 -> xyz=0.42 0.27 0.66 rpy=0 0 0.7854
- joint front_left_knee: axis 1 0 0 -> 0 1 0; limit lower=-2.35 upper=0.25 effort=38 velocity=3.5 -> lower=-1.5 upper=1.1 effort=42 velocity=3.5; origin xyz=0 0.39 -0.18 rpy=0 0 0 -> xyz=0.40 0 0 rpy=0 1.0 0
- joint front_right_hip_pitch: axis 1 0 0 -> 0 1 0; limit lower=-1.15 upper=1.15 effort=34 velocity=3 -> lower=-0.85 upper=1.05 effort=38 velocity=3; origin xyz=0 -0.2 0 rpy=0 0 0 -> xyz=0.22 0 0 rpy=0 0.52 0
- joint front_right_hip_yaw: limit lower=-0.8 upper=0.8 effort=28 velocity=3 -> lower=-0.75 upper=0.75 effort=30 velocity=3; origin xyz=0.46 -0.3 0 rpy=0 0 0 -> xyz=0.42 -0.27 0.66 rpy=0 0 -0.7854
- joint front_right_knee: axis 1 0 0 -> 0 1 0; limit lower=-2.35 upper=0.25 effort=38 velocity=3.5 -> lower=-1.5 upper=1.1 effort=42 velocity=3.5; origin xyz=0 -0.39 -0.18 rpy=0 0 0 -> xyz=0.40 0 0 rpy=0 1.0 0
- joint middle_left_hip_pitch: axis 1 0 0 -> 0 1 0; limit lower=-1.15 upper=1.15 effort=34 velocity=3 -> lower=-0.85 upper=1.05 effort=38 velocity=3; origin xyz=0 0.2 0 rpy=0 0 0 -> xyz=0.22 0 0 rpy=0 0.52 0
- joint middle_left_hip_yaw: limit lower=-0.8 upper=0.8 effort=28 velocity=3 -> lower=-0.75 upper=0.75 effort=30 velocity=3; origin xyz=0 0.34 0 rpy=0 0 0 -> xyz=0 0.29 0.66 rpy=0 0 1.5708
- joint middle_left_knee: axis 1 0 0 -> 0 1 0; limit lower=-2.35 upper=0.25 effort=38 velocity=3.5 -> lower=-1.5 upper=1.1 effort=42 velocity=3.5; origin xyz=0 0.39 -0.18 rpy=0 0 0 -> xyz=0.40 0 0 rpy=0 1.0 0
- joint middle_right_hip_pitch: axis 1 0 0 -> 0 1 0; limit lower=-1.15 upper=1.15 effort=34 velocity=3 -> lower=-0.85 upper=1.05 effort=38 velocity=3; origin xyz=0 -0.2 0 rpy=0 0 0 -> xyz=0.22 0 0 rpy=0 0.52 0
- joint middle_right_hip_yaw: limit lower=-0.8 upper=0.8 effort=28 velocity=3 -> lower=-0.75 upper=0.75 effort=30 velocity=3; origin xyz=0 -0.34 0 rpy=0 0 0 -> xyz=0 -0.29 0.66 rpy=0 0 -1.5708
- joint middle_right_knee: axis 1 0 0 -> 0 1 0; limit lower=-2.35 upper=0.25 effort=38 velocity=3.5 -> lower=-1.5 upper=1.1 effort=42 velocity=3.5; origin xyz=0 -0.39 -0.18 rpy=0 0 0 -> xyz=0.40 0 0 rpy=0 1.0 0
- joint rear_left_hip_pitch: axis 1 0 0 -> 0 1 0; limit lower=-1.15 upper=1.15 effort=34 velocity=3 -> lower=-0.85 upper=1.05 effort=38 velocity=3; origin xyz=0 0.2 0 rpy=0 0 0 -> xyz=0.22 0 0 rpy=0 0.52 0
- joint rear_left_hip_yaw: limit lower=-0.8 upper=0.8 effort=28 velocity=3 -> lower=-0.75 upper=0.75 effort=30 velocity=3; origin xyz=-0.46 0.3 0 rpy=0 0 0 -> xyz=-0.42 0.27 0.66 rpy=0 0 2.3562
- joint rear_left_knee: axis 1 0 0 -> 0 1 0; limit lower=-2.35 upper=0.25 effort=38 velocity=3.5 -> lower=-1.5 upper=1.1 effort=42 velocity=3.5; origin xyz=0 0.39 -0.18 rpy=0 0 0 -> xyz=0.40 0 0 rpy=0 1.0 0
- joint rear_right_hip_pitch: axis 1 0 0 -> 0 1 0; limit lower=-1.15 upper=1.15 effort=34 velocity=3 -> lower=-0.85 upper=1.05 effort=38 velocity=3; origin xyz=0 -0.2 0 rpy=0 0 0 -> xyz=0.22 0 0 rpy=0 0.52 0
- joint rear_right_hip_yaw: limit lower=-0.8 upper=0.8 effort=28 velocity=3 -> lower=-0.75 upper=0.75 effort=30 velocity=3; origin xyz=-0.46 -0.3 0 rpy=0 0 0 -> xyz=-0.42 -0.27 0.66 rpy=0 0 -2.3562
- joint rear_right_knee: axis 1 0 0 -> 0 1 0; limit lower=-2.35 upper=0.25 effort=38 velocity=3.5 -> lower=-1.5 upper=1.1 effort=42 velocity=3.5; origin xyz=0 -0.39 -0.18 rpy=0 0 0 -> xyz=0.40 0 0 rpy=0 1.0 0

File: assets/examples/turtle-style-bot/turtle-style-bot.urdf (robot description, URDF)
Before this commit: robot turtle_style_bot, 8 links, 7 joints
Links:
- removed link base_footprint
- removed link front_camera
- removed link sensor_mast
- added link camera_link, mass 0.14; collision box size=0.065 0.15 0.055; visual box size=0.065 0.15 0.055
- added link camera_mount, mass 0.08; collision box size=0.035 0.035 0.11; visual box size=0.035 0.035 0.11
- added link front_caster, mass 0.05; collision sphere radius=0.025; visual sphere radius=0.025
- added link imu_link, mass 0.03; collision box size=0.045 0.035 0.012; visual box size=0.045 0.035 0.012
- added link sensor_platform, mass 0.62; collision box size=0.255 0.255 0.018; visual box size=0.145 0.12 0.055
- link base_link: mass 5.2 -> 2.8; geometry collision cylinder length=0.15 radius=0.17; visual box size=0.018 0.165 0.055
- link left_wheel: mass 0.42 -> 0.23; geometry collision cylinder length=0.032 radius=0.066; visual cylinder length=0.032 radius=0.066
- link lidar_link: mass 0.22 -> 0.16; geometry collision cylinder length=0.076 radius=0.055; visual cylinder length=0.018 radius=0.049
- link rear_caster: mass 0.08 -> 0.05; geometry collision sphere radius=0.025; visual sphere radius=0.025
- link right_wheel: mass 0.42 -> 0.23; geometry collision cylinder length=0.032 radius=0.066; visual cylinder length=0.032 radius=0.066
Joints:
- removed joint base_joint
- removed joint camera_joint
- removed joint mast_joint
- added joint camera_mount_joint: type fixed, parent sensor_platform, child camera_mount, origin xyz=0.09 0 0.18 rpy=0 0 0
- added joint camera_tilt_joint: type revolute, parent camera_mount, child camera_link, origin xyz=0 0 0.125 rpy=0 0 0, axis 0 1 0, limit lower=-0.8 upper=0.45 effort=2 velocity=1.5
- added joint front_caster_joint: type fixed, parent base_link, child front_caster, origin xyz=0.125 0 0.025 rpy=0 0 0
- added joint imu_joint: type fixed, parent base_link, child imu_link, origin xyz=-0.055 0 0.13 rpy=0 0 0
- added joint sensor_platform_joint: type fixed, parent base_link, child sensor_platform, origin xyz=0 0 0.15 rpy=0 0 0
- joint left_wheel_joint: limit effort=12 velocity=12 -> effort=8 velocity=12; origin xyz=0 0.325 0.085 rpy=0 0 0 -> xyz=0 0.178 0.066 rpy=0 0 0
- joint lidar_joint: limit effort=1 velocity=8 -> effort=1 velocity=10; origin xyz=0 0 0.275 rpy=0 0 0 -> xyz=0 0 0.18 rpy=0 0 0; parent sensor_mast -> sensor_platform
- joint rear_caster_joint: origin xyz=-0.235 0 -0.055 rpy=0 0 0 -> xyz=-0.125 0 0.025 rpy=0 0 0
- joint right_wheel_joint: limit effort=12 velocity=12 -> effort=8 velocity=12; origin xyz=0 -0.325 0.085 rpy=0 0 0 -> xyz=0 -0.178 0.066 rpy=0 0 0
